File: docs/martinez.sch (EAGLE design)
At the start: 52 parts, among them IC2 LM3480-3.3V, Q1 BSS138, Q2 BSS138, X2 USBOLD, Y7 16mhz

Commit message: new eagle board
Parts:
- removed JP2: (no value), SparkFun:M05PTH
- removed JP3: (no value), SparkFun:M081X08
- removed JP4: M09, SparkFun:M09
- added J1: AVR_SPI_PRG_6PTH, SparkFun:AVR_SPI_PRG_6PTH
- added JP10, JP8: (no value), SparkFun:M031X03_NO_SILK
- added JP11: (no value), SparkFun:M041X04_NO_SILK
- added JP5: (no value), SparkFun:M05PTH
- F1: value FUSE_SMD_10MM -> OMT125_4A; device f-lf-omniblok-s:FUSE_SMD_10MM -> fuse:OMT125_11MM
Connections:
- net +5V: now also J1.2, JP10.2, JP11.3, JP5.1; no longer JP2.1, JP4.1
- net A1: now also JP8.2; no longer JP3.2
- net A2: now also JP8.1; no longer JP3.1
- net CH2: no longer JP3.6
- net CH3: no longer JP3.5
- net GND: now also J1.6, JP10.3, JP11.4, JP5.4, JP8.3; no longer JP2.5, JP3.3, JP3.8, JP4.3
- net INT: now also JP5.5; no longer JP2.4, JP3.7
- net MISO: now also J1.1; no longer JP3.4
- net MOSI/PWM6: now also J1.4; no longer JP4.4
- net MULTI_PORT: now also JP10.1; no longer JP4.2
- net RESET: now also J1.5; no longer JP4.6
- net RXD: now also JP11.2; no longer JP4.7
- net SCK_EN: now also J1.3; no longer JP4.5
- net SCL_3V: now also JP5.3; no longer JP2.3
- net SDA_3V: now also JP5.2; no longer JP2.2
- net TXD: now also JP11.1; no longer JP4.8
- net VCC: no longer JP4.9
